Commit message: Added tof ring config in ur model

File: urdf/ur.urdf.xacro (robot description, xacro)
@@ -5,7 +5,10 @@
    <!-- import main macro -->
    <xacro:include filename="$(find ur_description)/urdf/ur_macro.xacro"/>
+   <!-- sensors macros (also add flat flange) -->
+   <xacro:include filename="$(find proxysim_description)/urdf/common_properties.xacro" />
+   <xacro:include filename="$(find proxysim_description)/urdf/tof_ring_parametric.xacro"/>
    <!-- possible 'ur_type' values: ur3, ur3e, ur5, ur5e, ur10, ur10e, ur16e, ur20, ur30 -->
    <!-- the default value should raise an error in case this was called without defining the type -->
-   <xacro:arg name="ur_type" default="ur5x"/>
+   <xacro:arg name="ur_type" default="ur10e"/>
    <!-- parameters -->
    <xacro:arg name="tf_prefix" default="" />
@@ -89,6 +92,16 @@
      trajectory_port="$(arg trajectory_port)"
      >
-     <origin xyz="0 0 0" rpy="0 0 0" />          <!-- position robot in the world -->
+     <origin xyz="0 0 0" rpy="0 0 0" />   <!-- position robot in the world -->
    </xacro:ur_robot>
+   <!-- sensors -->
+   <xacro:tof_ring
+    array_name="tof_ring_0"
+    root_link="shoulder_link"
+    x="0"
+    y="0"
+    z="0"
+    roll="0"
+    pitch="0"
+    yaw="0"/>
    <xacro:if value="$(arg sim_gazebo)">
     <!-- Gazebo plugins -->
