Commit message: adjusted range for simulated measurements

File: urdf/ur_flange_tof.urdf.xacro (robot description, xacro)
@@ -95,5 +95,5 @@
      trajectory_port="$(arg trajectory_port)"
      >
-     <origin xyz="0 0 0" rpy="0 0 0" />   <!-- position robot in the world -->
+     <origin xyz="0 0 0.02" rpy="0 0 0" />   <!-- position robot in the world - small offset on z to avoid floor collision -->
    </xacro:ur_robot>
     <!-- Sensors -->

File: urdf/ur_flange_tof_imu.urdf.xacro (robot description, xacro)
@@ -9,4 +9,5 @@
    <xacro:include filename="$(find proxysim_description)/urdf/tof_ring_parametric.xacro"/>
    <xacro:include filename="$(find proxysim_description)/urdf/tof_sensor_parametric.xacro"/>
+   <xacro:include filename="$(find proxysim_description)/urdf/imu_sensor_parametric.xacro"/>
    <!-- custom models macros -->
    <xacro:include filename="$(find ur_proxysim_description)/urdf/calibration_plane.xacro"/>
@@ -97,5 +98,5 @@
      <origin xyz="0 0 0" rpy="0 0 0" />   <!-- position robot in the world -->
    </xacro:ur_robot>
-   <!-- Sensors -->
+  <!-- Sensors -->
   <!-- flange tof sensor -->
   <xacro:tof_sensor
@@ -110,4 +111,14 @@
   </xacro:tof_sensor>
   <!-- flange imu sensor -->
+  <xacro:imu_sensor
+  tf_prefix="ur_ee_imu"
+  base_link="wrist_2_link"
+  x="0"
+  y="0"
+  z="0"
+  roll="0"
+  pitch="0"
+  yaw="0">
+  </xacro:imu_sensor>
    <xacro:if value="$(arg sim_gazebo)">
     <!-- Gazebo plugins -->
